File: pcb/es8156_breakout.kicad_sch (KiCad schematic)
At the start: 9 parts, among them CN1 PJ-320D, J2 Conn_01x12, J3 Conn_01x03, U1 ES8156

Commit message: update schematic & pcb
Parts:
- removed C1, C2, C3, C4: 1u, Capacitor_SMD:C_0603_1608Metric_Pad1.08x0.95mm_HandSolder, symbol Device:C
- removed C5: 100n, Capacitor_SMD:C_0603_1608Metric_Pad1.08x0.95mm_HandSolder, symbol Device:C
- removed J2: Conn_01x12, Connector_PinHeader_2.54mm:PinHeader_1x12_P2.54mm_Vertical, symbol Connector_Generic:Conn_01x12
- added C1, C2, C3, C4, C5: 1u, Capacitor_SMD:C_0603_1608Metric_Pad1.08x0.95mm_HandSolder, symbol Device:C_Small
- added J1: Conn_01x08, Connector_PinHeader_2.54mm:PinHeader_1x08_P2.54mm_Vertical, symbol Connector_Generic:Conn_01x08
- added R1: 10k, Resistor_SMD:R_0603_1608Metric_Pad0.98x0.95mm_HandSolder, symbol Device:R_Small
- added R2, R3: 33R, Resistor_SMD:R_0603_1608Metric_Pad0.98x0.95mm_HandSolder, symbol Device:R_Small
- renumbered J3 to J2
Connections:
- net VD is gone; now on net VALL: U1.4 (DVDD)
- net VP is gone; now on net VALL: U1.5 (PVDD)
- net CCLK: now also J1.4 (Pin_4)
- net CDATA: now also J1.3 (Pin_3)
- net GND: now also C1.2, C2.2, C3.1, C4.1, C5.1, J1.1 (Pin_1), R1.1
- net HPCOM: now also CN1.1
- net LRCK: now also J1.8 (Pin_8)
- net Left: now also J2.2 (Pin_2), R2.1; no longer CN1.4, J2.3 (Pin_3)
- net MCLK: now also J1.5 (Pin_5)
- net Right: now also J2.3 (Pin_3), R3.1; no longer CN1.3, J2.2 (Pin_2)
- net SCLK: now also J1.6 (Pin_6)
- net SDIN: now also J1.7 (Pin_7)
- net at U1.17 (VRP): now also C4.2
- net at U1.18 (VMID): now also C3.2
- net CE: no longer names the net of U1.19 (CE)
- net CE: now also R1.2
- net SDOUT: no longer names the net of U1.20 (SDOUT)
- net VA renamed VALL
- net VALL: now also C1.1, C2.1, C5.2, J1.2 (Pin_2)
- new net HP_Left: CN1.4, R2.2
- new net HP_Right: CN1.3, R3.2
Other:
- moved on the sheet: CN1, J2
